File: 0.1/greenpill.sch (KiCad schematic (older format))
At the start: 31 parts, among them J1 Conn_01x20_Male, J2 Conn_01x20_Male, J3 Conn_01x04_Male, J5 USB_C_Receptacle_USB2.0, SW1 SW_Push, SW2 SW_Push, U1 ATSAMD51G18A-M, U2 MIC5504-3.3YM5, U3 S25FL064, Y1 Crystal_GND23

Commit message: PINOUT CHANGE, rerouted and updated silk.s
Swapped left pins 13 and 16 (formerly A21 & A27 respectively) so PWM output on A21 can be used for Textier LED4:G. A27 now on pin L13 is used for key matrix scanning and so doesn't require PWM
Rerouted only affected traces
Swapped silkscreen labels
Connections:
- net pa21: now also J1.16 (Pin_16); no longer J1.13 (Pin_13)
- net pa27: now also J1.13 (Pin_13); no longer J1.16 (Pin_16)
Changed lines of the file:
@@
 Wire Wire Line
 	7850 3050 8050 3050
-Text Label 8050 3150 2    50   ~ 0
+Text Label 8050 2850 2    50   ~ 0
 pa27
 Wire Wire Line
@@
 Wire Wire Line
 	7850 2850 8050 2850
-Text Label 8050 2850 2    50   ~ 0
+Text Label 8050 3150 2    50   ~ 0
 pa21
 Text Label 8750 3550 2    50   ~ 0

Commit message: a bit of tweaking
Parts:
- C7, C8: value 1u -> 10u
Connections:
- net pa02: now also R6.2, SW2.1
- net pb02: no longer R6.2, SW2.1
Other:
- moved on the sheet: C7, C8
Changed lines of the file:
@@
 L power:+3V3 #PWR0128
 U 1 1 5F092C58
-P 2100 1650
-F 0 "#PWR0128" H 2100 1500 50  0001 C CNN
-F 1 "+3V3" H 2115 1823 50  0000 C CNN
-F 2 "" H 2100 1650 50  0001 C CNN
-F 3 "" H 2100 1650 50  0001 C CNN
-	1    2100 1650
+P 2100 1700
+F 0 "#PWR0128" H 2100 1550 50  0001 C CNN
+F 1 "+3V3" H 2115 1873 50  0000 C CNN
+F 2 "" H 2100 1700 50  0001 C CNN
+F 3 "" H 2100 1700 50  0001 C CNN
+	1    2100 1700
 	1    0    0    -1
 $EndComp
@@
 L Device:C_Small C8
 U 1 1 5F094026
-P 2100 1750
-F 0 "C8" H 2192 1796 50  0000 L CNN
-F 1 "1u" H 2192 1705 50  0000 L CNN
-F 2 "Capacitor_SMD:C_0603_1608Metric" H 2100 1750 50  0001 C CNN
-F 3 "~" H 2100 1750 50  0001 C CNN
-	1    2100 1750
+P 2100 1800
+F 0 "C8" H 2192 1846 50  0000 L CNN
+F 1 "10u" H 2192 1755 50  0000 L CNN
+F 2 "Capacitor_SMD:C_0603_1608Metric" H 2100 1800 50  0001 C CNN
+F 3 "~" H 2100 1800 50  0001 C CNN
+	1    2100 1800
 	1    0    0    -1
 $EndComp
@@
 L Device:C_Small C7
 U 1 1 5F094AF2
-P 1000 1750
-F 0 "C7" H 1092 1796 50  0000 L CNN
-F 1 "1u" H 1092 1705 50  0000 L CNN
-F 2 "Capacitor_SMD:C_0603_1608Metric" H 1000 1750 50  0001 C CNN
-F 3 "~" H 1000 1750 50  0001 C CNN
-	1    1000 1750
+P 1000 1800
+F 0 "C7" H 1092 1846 50  0000 L CNN
+F 1 "10u" H 1092 1755 50  0000 L CNN
+F 2 "Capacitor_SMD:C_0603_1608Metric" H 1000 1800 50  0001 C CNN
+F 3 "~" H 1000 1800 50  0001 C CNN
+	1    1000 1800
 	1    0    0    -1
 $EndComp
@@
 L power:GND #PWR0129
 U 1 1 5F0A028B
-P 2100 1850
-F 0 "#PWR0129" H 2100 1600 50  0001 C CNN
-F 1 "GND" H 2105 1677 50  0000 C CNN
-F 2 "" H 2100 1850 50  0001 C CNN
-F 3 "" H 2100 1850 50  0001 C CNN
-	1    2100 1850
+P 2100 1900
+F 0 "#PWR0129" H 2100 1650 50  0001 C CNN
+F 1 "GND" H 2105 1727 50  0000 C CNN
+F 2 "" H 2100 1900 50  0001 C CNN
+F 3 "" H 2100 1900 50  0001 C CNN
+	1    2100 1900
 	1    0    0    -1
 $EndComp
@@
 L power:GND #PWR0130
 U 1 1 5F0A0A87
-P 1000 1850
-F 0 "#PWR0130" H 1000 1600 50  0001 C CNN
-F 1 "GND" H 1005 1677 50  0000 C CNN
-F 2 "" H 1000 1850 50  0001 C CNN
-F 3 "" H 1000 1850 50  0001 C CNN
-	1    1000 1850
+P 1000 1900
+F 0 "#PWR0130" H 1000 1650 50  0001 C CNN
+F 1 "GND" H 1005 1727 50  0000 C CNN
+F 2 "" H 1000 1900 50  0001 C CNN
+F 3 "" H 1000 1900 50  0001 C CNN
+	1    1000 1900
 	1    0    0    -1
 $EndComp
@@
 L power:+5V #PWR0131
 U 1 1 5F0A152D
-P 1000 1650
-F 0 "#PWR0131" H 1000 1500 50  0001 C CNN
-F 1 "+5V" H 1015 1823 50  0000 C CNN
-F 2 "" H 1000 1650 50  0001 C CNN
-F 3 "" H 1000 1650 50  0001 C CNN
-	1    1000 1650
+P 1000 1700
+F 0 "#PWR0131" H 1000 1550 50  0001 C CNN
+F 1 "+5V" H 1015 1873 50  0000 C CNN
+F 2 "" H 1000 1700 50  0001 C CNN
+F 3 "" H 1000 1700 50  0001 C CNN
+	1    1000 1700
 	1    0    0    -1
 $EndComp
@@
 	5050 2300 5850 2300
 Text Label 5850 2400 2    50   ~ 0
-pb02
+pa02
 Text Label 5850 2300 2    50   ~ 0
 pb09

Commit message: Switched to QFN-64 package, reassigned pins. Trimmed Edge.Cuts
Still TODO:
 - Redo silkscreen
 - Move passives near MCU to optimal position (1v2 caps especially)
Parts:
- removed U1: ATSAMD51G18A-M, Package_DFN_QFN:QFN-48-1EP_7x7mm_P0.5mm_EP5.15x5.15mm, symbol greenpill:ATSAMD51G18A-M
- added U1: ATSAMD51J18A-M, Package_DFN_QFN:QFN-64-1EP_9x9mm_P0.5mm_EP4.7x4.7mm, symbol MCU_Microchip_SAMD:ATSAMD51J18A-M
Connections:
- net !reset: now also U1.52 (~RESET)
- net +1V2: now also U1.53 (VDDCORE)
- net +3V3: now also U1.21 (VDDIOB), U1.34 (VDDIO), U1.48 (VDDIO), U1.56 (VDDIO)
- net GND: now also U1.22 (GND), U1.33 (GND), U1.47 (GND), U1.54 (GND), U1.65 (GND), U1.7 (GNDANA)
- net pa00: now also U1.1 (PA00)
- net pa01: now also U1.2 (PA01)
- net pa02: now also J2.15 (Pin_15), U1.3 (PA02); no longer J2.19 (Pin_19)
- net pa03: now also U1.4 (PA03)
- net pa04: now also U1.13 (PA04)
- net pa05: now also U1.14 (PA05)
- net pa06: now also U1.15 (PA06)
- net pa07: now also U1.16 (PA07)
- net pa08: now also U1.17 (PA08)
- net pa09: now also U1.18 (PA09)
- net pa10: now also U1.19 (PA10)
- net pa11: now also U1.20 (PA11); no longer J2.7 (Pin_7)
- net pa12: now also U1.29 (PA12); no longer J2.4 (Pin_4)
- net pa13: now also U1.30 (PA13); no longer J1.1 (Pin_1)
- net pa14: now also U1.31 (PA14); no longer J1.2 (Pin_2)
- net pa15: now also U1.32 (PA15); no longer J1.3 (Pin_3)
- net pa16: now also J1.1 (Pin_1), U1.35 (PA16); no longer J1.4 (Pin_4)
- net pa17: now also J1.2 (Pin_2), U1.36 (PA17); no longer J1.5 (Pin_5)
- net pa18: now also J1.3 (Pin_3), U1.37 (PA18); no longer J1.6 (Pin_6)
- net pa19: now also J1.4 (Pin_4), U1.38 (PA19); no longer J1.7 (Pin_7)
- net pa20: now also J1.7 (Pin_7), U1.41 (PA20); no longer J1.10 (Pin_10)
- net pa21: now also U1.42 (PA21); no longer J1.16 (Pin_16)
- net pa22: now also J1.10 (Pin_10), U1.43 (PA22); no longer J1.12 (Pin_12)
- net pa23: now also U1.44 (PA23); no longer J1.11 (Pin_11)
- net pa24: now also U1.45 (PA24)
- net pa25: now also U1.46 (PA25)
- net pa27: now also U1.51 (PA27)
- net pa30: now also U1.57 (PA30)
- net pa31: now also U1.58 (PA31)
- net pb02: now also U1.63 (PB02)
- net pb03: now also U1.64 (PB03)
- net pb08: now also U1.11 (PB08); no longer J2.17 (Pin_17)
- net pb09: now also U1.12 (PB09); no longer D2.2 (A), J2.15 (Pin_15)
- net pb10: now also J2.7 (Pin_7), U1.23 (PB10); no longer J2.6 (Pin_6)
- net pb11: now also J2.6 (Pin_6), U1.24 (PB11); no longer J2.5 (Pin_5)
- net pb22: now also J1.11 (Pin_11), U1.49 (PB22); no longer J1.14 (Pin_14)
- net pb23: now also J1.12 (Pin_12), U1.50 (PB23); no longer J1.15 (Pin_15)
- net vsw: now also U1.55 (VSW)
- new net pb00: J1.15 (Pin_15), U1.61 (PB00)
- new net pb01: J1.16 (Pin_16), U1.62 (PB01)
- new net pb04: D2.2 (A), J2.19 (Pin_19), U1.5 (PB04)
- new net pb05: U1.6 (PB05)
- new net pb06: U1.9 (PB06)
- new net pb07: U1.10 (PB07)
- new net pb12: J2.5 (Pin_5), U1.25 (PB12)
- new net pb13: J2.4 (Pin_4), U1.26 (PB13)
- new net pb14: U1.27 (PB14)
- new net pb15: U1.28 (PB15)
- new net pb16: J1.5 (Pin_5), U1.39 (PB16)
- new net pb17: J1.6 (Pin_6), U1.40 (PB17)
- new net pb30: J2.17 (Pin_17), U1.59 (PB30)
- new net pb31: J1.14 (Pin_14), U1.60 (PB31)
Other:
- note added: "TODO: \nwork out if/why SAMD51\n needs BOOT0 button"
- note added: "TODO\nReassign sercom to pins \nthat aren't broken out"
- note added: "pb30 has tcc0 \nfor neopixel DMA"
- moved on the sheet: D1, D2, J1, J2, J3, R3, R4, R5, R6, SW1, SW2

Commit message: swapped button and led to non broken out pins
Connections:
- net pa02: no longer R6.2, SW2.1
- net pb04: no longer D2.2 (A)
- net pb06: now also R6.2, SW2.1
- net pb08: now also D2.2 (A)
Changed lines of the file:
@@
 TODO: \nwork out if/why SAMD51\n needs BOOT0 button
 Text Label 8400 3000 0    50   ~ 0
-user_button
+pa02
 Text Label 1950 3200 0    50   ~ 0
 usb_d-
@@
 pb02
 Text Label 8400 3400 0    50   ~ 0
-user_led
+pb04
 Text Label 8400 3200 0    50   ~ 0
 pb30
@@
 pa14
 Text Label 5850 2300 2    50   ~ 0
-pb04
+pb08
 Text Label 5850 2400 2    50   ~ 0
-pa02
+pb06
 $EndSCHEMATC

Commit message: add mpns
Parts:
- C1, C10, C2, C3, C4, C6, C9: MPN (none) -> GRM155R61A104KA01J
- C11, C12: MPN (none) -> C0603C120J5GACTU
- C5: MPN (none) -> CL10A475KQ8NNNC
- C7, C8: MPN (none) -> GRM188R61A106KE69J
- D1: MPN (none) -> 150060RS75000
- D2: MPN (none) -> 150060BS75000
- D3: MPN (none) -> BAT54C,215
- J5: MPN (none) -> lmao aliexpress
- R1, R2: MPN (none) -> RC0603FR-075K1L
- R3: value R_Small -> 261; MPN (none) -> P261HCT-ND
- R4: value R_Small -> 60.4; MPN (none) -> RC0603FR-0760R4L
- R5, R6: MPN (none) -> RC0603FR-0710KL
- SW1, SW2: MPN (none) -> PTS815 SJM 250 SMTR LFS
- U1: value ATSAMD51J18A-M -> ATSAMD51J20A-M; symbol MCU_Microchip_SAMD:ATSAMD51J18A-M -> MCU_Microchip_SAMD:ATSAMD51J20A-M; MPN (none) -> ATSAMD51J20A-MU
- U2: MPN (none) -> MIC5504-3.3YM5-TR
- U3: MPN (none) -> S25FL064LABMFN010
- Y1: MPN (none) -> FC-135 32.7680KA-A5
Changed lines of the file:
@@
 F 2 "Capacitor_SMD:C_0402_1005Metric" H 2550 1150 50  0001 C CNN
 F 3 "~" H 2550 1150 50  0001 C CNN
+F 4 "GRM155R61A104KA01J" H 2550 1150 50  0001 C CNN "MPN"
 	1    2550 1150
 	1    0    0    -1
@@
 F 2 "Connector_USB:USB_C_Receptacle_XKB_U262-16XN-4BVC11" H 1500 3200 50  0001 C CNN
 F 3 "https://www.usb.org/sites/default/files/documents/usb_type-c.zip" H 1500 3200 50  0001 C CNN
+F 4 "lmao aliexpress" H 1350 3200 50  0001 C CNN "MPN"
 	1    1350 3200
 	1    0    0    -1
@@
 F 2 "Capacitor_SMD:C_0402_1005Metric" H 2900 1150 50  0001 C CNN
 F 3 "~" H 2900 1150 50  0001 C CNN
+F 4 "GRM155R61A104KA01J" H 2900 1150 50  0001 C CNN "MPN"
 	1    2900 1150
 	1    0    0    -1
@@
 F 2 "Capacitor_SMD:C_0402_1005Metric" H 3250 1150 50  0001 C CNN
 F 3 "~" H 3250 1150 50  0001 C CNN
+F 4 "GRM155R61A104KA01J" H 3250 1150 50  0001 C CNN "MPN"
 	1    3250 1150
 	1    0    0    -1
@@
 F 2 "Capacitor_SMD:C_0402_1005Metric" H 3650 1150 50  0001 C CNN
 F 3 "~" H 3650 1150 50  0001 C CNN
+F 4 "GRM155R61A104KA01J" H 3650 1150 50  0001 C CNN "MPN"
 	1    3650 1150
 	1    0    0    -1
@@
 F 2 "Capacitor_SMD:C_0402_1005Metric" H 2550 1800 50  0001 C CNN
 F 3 "~" H 2550 1800 50  0001 C CNN
+F 4 "GRM155R61A104KA01J" H 2550 1800 50  0001 C CNN "MPN"
 	1    2550 1800
 	1    0    0    -1
@@
 F 2 "Capacitor_SMD:C_0603_1608Metric" H 2950 1800 50  0001 C CNN
 F 3 "~" H 2950 1800 50  0001 C CNN
+F 4 "CL10A475KQ8NNNC" H 2950 1800 50  0001 C CNN "MPN"
 	1    2950 1800
 	1    0    0    -1
@@
 F 2 "Package_TO_SOT_SMD:SOT-23-5" H 1550 750 50  0001 C CNN
 F 3 "http://ww1.microchip.com/downloads/en/DeviceDoc/MIC550X.pdf" H 1300 1400 50  0001 C CNN
+F 4 "MIC5504-3.3YM5-TR" H 1550 1150 50  0001 C CNN "MPN"
 	1    1550 1150
 	1    0    0    -1
@@
 F 2 "Capacitor_SMD:C_0603_1608Metric" H 2100 1800 50  0001 C CNN
 F 3 "~" H 2100 1800 50  0001 C CNN
+F 4 "GRM188R61A106KE69J" H 2100 1800 50  0001 C CNN "MPN"
 	1    2100 1800
 	1    0    0    -1
@@
 F 2 "Capacitor_SMD:C_0603_1608Metric" H 1000 1800 50  0001 C CNN
 F 3 "~" H 1000 1800 50  0001 C CNN
+F 4 "GRM188R61A106KE69J" H 1000 1800 50  0001 C CNN "MPN"
 	1    1000 1800
 	1    0    0    -1
@@
 F 2 "Resistor_SMD:R_0603_1608Metric" H 2400 2850 50  0001 C CNN
 F 3 "~" H 2400 2850 50  0001 C CNN
+F 4 "RC0603FR-075K1L" H 2400 2850 50  0001 C CNN "MPN"
 	1    2400 2850
 	-1   0    0    1
@@
 F 2 "Resistor_SMD:R_0603_1608Metric" H 2700 2850 50  0001 C CNN
 F 3 "~" H 2700 2850 50  0001 C CNN
+F 4 "RC0603FR-075K1L" H 2700 2850 50  0001 C CNN "MPN"
 	1    2700 2850
 	1    0    0    -1
@@
 F 1 "LED" H 6793 3026 50  0000 C CNN
 F 2 "LED_SMD:LED_0603_1608Metric" H 6800 2900 50  0001 C CNN
-F 3 "~" H 6800 2900 50  0001 C CNN
+F 3 "https://www.we-online.de/katalog/datasheet/150060RS75000.pdf" H 6800 2900 50  0001 C CNN
+F 4 "150060RS75000" H 6800 2900 50  0001 C CNN "MPN"
 	1    6800 2900
 	1    0    0    -1
@@
 F 1 "LED" H 6793 3426 50  0000 C CNN
 F 2 "LED_SMD:LED_0603_1608Metric" H 6800 3300 50  0001 C CNN
-F 3 "~" H 6800 3300 50  0001 C CNN
+F 3 "https://www.we-online.de/katalog/datasheet/150060BS75000.pdf" H 6800 3300 50  0001 C CNN
+F 4 "150060BS75000" H 6800 3300 50  0001 C CNN "MPN"
 	1    6800 3300
 	1    0    0    -1
@@
 P 6550 2900
 F 0 "R3" V 6354 2900 50  0000 C CNN
-F 1 "R_Small" V 6445 2900 50  0000 C CNN
+F 1 "261" V 6445 2900 50  0000 C CNN
 F 2 "Resistor_SMD:R_0603_1608Metric" H 6550 2900 50  0001 C CNN
 F 3 "~" H 6550 2900 50  0001 C CNN
+F 4 "P261HCT-ND" V 6550 2900 50  0001 C CNN "MPN"
 	1    6550 2900
 	0    1    1    0
@@
 P 6550 3300
 F 0 "R4" V 6354 3300 50  0000 C CNN
-F 1 "R_Small" V 6445 3300 50  0000 C CNN
+F 1 "60.4" V 6445 3300 50  0000 C CNN
 F 2 "Resistor_SMD:R_0603_1608Metric" H 6550 3300 50  0001 C CNN
 F 3 "~" H 6550 3300 50  0001 C CNN
+F 4 "RC0603FR-0760R4L" V 6550 3300 50  0001 C CNN "MPN"
 	1    6550 3300
 	0    1    1    0
@@
 F 1 "SW_Push" H 6750 5394 50  0000 C CNN
 F 2 "greenpill:pts815" H 6750 5400 50  0001 C CNN
-F 3 "~" H 6750 5400 50  0001 C CNN
+F 3 "" H 6750 5400 50  0001 C CNN
+F 4 "PTS815 SJM 250 SMTR LFS" H 6750 5200 50  0001 C CNN "MPN"
 	1    6750 5200
 	1    0    0    -1
@@
 F 1 "SW_Push" H 6750 5844 50  0000 C CNN
 F 2 "greenpill:pts815" H 6750 5850 50  0001 C CNN
-F 3 "~" H 6750 5850 50  0001 C CNN
+F 3 "" H 6750 5850 50  0001 C CNN
+F 4 "PTS815 SJM 250 SMTR LFS" H 6750 5650 50  0001 C CNN "MPN"
 	1    6750 5650
 	1    0    0    -1
@@
 F 2 "Package_TO_SOT_SMD:SOT-23" H 8025 4575 50  0001 L CNN
 F 3 "http://www.diodes.com/_files/datasheets/ds11005.pdf" H 7870 4450 50  0001 C CNN
+F 4 "BAT54C,215" H 7950 4450 50  0001 C CNN "MPN"
 	1    7950 4450
 	-1   0    0    1
@@
 F 2 "Capacitor_SMD:C_0402_1005Metric" H 8150 4150 50  0001 C CNN
 F 3 "~" H 8150 4150 50  0001 C CNN
+F 4 "GRM155R61A104KA01J" V 8150 4150 50  0001 C CNN "MPN"
 	1    8150 4150
 	0    1    1    0
@@
 F 2 "Capacitor_SMD:C_0402_1005Metric" H 4550 1100 50  0001 C CNN
 F 3 "~" H 4550 1100 50  0001 C CNN
+F 4 "GRM155R61A104KA01J" H 4550 1100 50  0001 C CNN "MPN"
 	1    4550 1100
 	1    0    0    -1
@@
 F 2 "Resistor_SMD:R_0603_1608Metric" H 6300 5550 50  0001 C CNN
 F 3 "~" H 6300 5550 50  0001 C CNN
+F 4 "RC0603FR-0710KL" H 6300 5550 50  0001 C CNN "MPN"
 	1    6300 5550
 	1    0    0    -1
@@
 F 2 "Resistor_SMD:R_0603_1608Metric" H 6300 5100 50  0001 C CNN
 F 3 "~" H 6300 5100 50  0001 C CNN
+F 4 "RC0603FR-0710KL" H 6300 5100 50  0001 C CNN "MPN"
 	1    6300 5100
 	1    0    0    -1
@@
 F 2 "Package_SO:SOIC-8_5.23x5.23mm_P1.27mm" H 5950 1050 50  0001 C CNN
 F 3 "" H 5950 1050 50  0001 C CNN
+F 4 "S25FL064LABMFN010" H 5950 1250 50  0001 C CNN "MPN"
 	1    5950 1250
 	1    0    0    -1
@@
 F 2 "Crystal:Crystal_SMD_3215-2Pin_3.2x1.5mm" H 7950 5100 50  0001 C CNN
 F 3 "~" H 7950 5100 50  0001 C CNN
+F 4 "FC-135 32.7680KA-A5" H 7950 5100 50  0001 C CNN "MPN"
 	1    7950 5100
 	1    0    0    -1
@@
 F 1 "12p" H 8292 5355 50  0000 L CNN
 F 2 "Capacitor_SMD:C_0603_1608Metric" H 8200 5400 50  0001 C CNN
-F 3 "~" H 8200 5400 50  0001 C CNN
+F 3 "" H 8200 5400 50  0001 C CNN
+F 4 "C0603C120J5GACTU" H 8200 5400 50  0001 C CNN "MPN"
 	1    8200 5400
 	1    0    0    -1
@@
 F 2 "Capacitor_SMD:C_0603_1608Metric" H 7700 5400 50  0001 C CNN
 F 3 "~" H 7700 5400 50  0001 C CNN
+F 4 "C0603C120J5GACTU" H 7700 5400 50  0001 C CNN "MPN"
 	1    7700 5400
 	1    0    0    -1
@@
 	5050 2300 5850 2300
 $Comp
-L MCU_Microchip_SAMD:ATSAMD51J18A-M U1
+L MCU_Microchip_SAMD:ATSAMD51J20A-M U1
 U 1 1 5F0167C3
 P 10050 3000
 F 0 "U1" H 10050 950 50  0000 C CNN
-F 1 "ATSAMD51J18A-M" H 10050 850 50  0000 C CNN
+F 1 "ATSAMD51J20A-M" H 10050 850 50  0000 C CNN
 F 2 "Package_DFN_QFN:QFN-64-1EP_9x9mm_P0.5mm_EP4.7x4.7mm" H 10050 3000 50  0001 C CIN
 F 3 "http://ww1.microchip.com/downloads/en/DeviceDoc/60001507E.pdf" H 10050 3000 50  0001 C CNN
+F 4 "ATSAMD51J20A-MU" H 10050 3000 50  0001 C CNN "MPN"
 	1    10050 3000
 	1    0    0    -1
