File: 1.0/greenpill.sch (KiCad schematic (older format))
At the start: 33 parts, among them J1 Conn_01x20_Male, J2 Conn_01x20_Male, J3 Conn_01x04_Male, J5 USB_C_Receptacle_USB2.0, SW1 SW_Push, SW2 SW_Push, U1 ATSAMD51J20A-M, U2 MIC5504-3.3YM5, U3 S25FL064, Y1 Crystal_GND23

Commit message: change pinout to hopefully have full timer coverage
Connections:
- net pa04: now also J2.10 (Pin_10); no longer J2.14 (Pin_14)
- net pa06: now also J2.11 (Pin_11); no longer J2.12 (Pin_12)
- net pa07: now also J2.12 (Pin_12); no longer J2.11 (Pin_11)
- net pa08: now also J2.14 (Pin_14); no longer J2.10 (Pin_10)
- net pa20: now also J1.10 (Pin_10); no longer J1.7 (Pin_7)
- net pa22: now also J1.15 (Pin_15); no longer J1.10 (Pin_10)
- net pb00: now also J1.7 (Pin_7); no longer J1.15 (Pin_15)
- net pb01: now also J1.6 (Pin_6); no longer J1.16 (Pin_16)
- net pb17: now also J1.16 (Pin_16); no longer J1.6 (Pin_6)
Changed lines of the file:
@@
 Text Label 7850 2400 2    50   ~ 0
 usb_d+
-Text Label 8400 2900 0    50   ~ 0
-pa04
-Text Label 8400 2800 0    50   ~ 0
-pa05
-Text Label 8400 2700 0    50   ~ 0
-pa06
-Text Label 8400 2600 0    50   ~ 0
-pa07
-Text Label 8400 2500 0    50   ~ 0
-pa08
-Text Label 8400 2400 0    50   ~ 0
-pa09
-Text Label 8400 2300 0    50   ~ 0
-pa10
-Text Label 8400 2200 0    50   ~ 0
-pb10
-Text Label 8400 2100 0    50   ~ 0
-pb11
-Text Label 8400 2000 0    50   ~ 0
-pb12
-Text Label 8400 1900 0    50   ~ 0
-pb13
 Text Label 7850 1600 2    50   ~ 0
 pa16
@@
 Text Label 9150 4100 2    50   ~ 0
 usb_d+
-Text Label 7850 2100 2    50   ~ 0
-pb17
-Text Label 7850 2200 2    50   ~ 0
-pa20
-Text Label 7850 2500 2    50   ~ 0
-pa22
 Text Label 7850 2600 2    50   ~ 0
 pb22
-Text Label 7850 2700 2    50   ~ 0
-pb23
-Text Label 7850 2800 2    50   ~ 0
-pa27
-Text Label 7850 2900 2    50   ~ 0
-pb31
-Text Label 7850 3000 2    50   ~ 0
-pb00
-Text Label 7850 3100 2    50   ~ 0
-pb01
-Text Label 7850 3200 2    50   ~ 0
-pb02
 Text Label 8400 3400 0    50   ~ 0
 pb04
@@
 	1150 1250 1150 1050
 Connection ~ 1150 1050
+$Comp
+L Graphic:Logo_Open_Hardware_Small #LOGO1
+U 1 1 5F548A14
+P 4750 3300
+F 0 "#LOGO1" H 4750 3575 50  0001 C CNN
+F 1 "Logo_Open_Hardware_Small" H 4750 3075 50  0001 C CNN
+F 2 "" H 4750 3300 50  0001 C CNN
+F 3 "~" H 4750 3300 50  0001 C CNN
+	1    4750 3300
+	1    0    0    -1
+$EndComp
+Text Label 7850 2800 2    50   ~ 0
+pa27
+Text Label 7850 2700 2    50   ~ 0
+pb23
+Text Label 7850 3000 2    50   ~ 0
+pa22
+Text Label 7850 2900 2    50   ~ 0
+pb31
+Text Label 7850 3200 2    50   ~ 0
+pb02
+Text Label 7850 2200 2    50   ~ 0
+pb00
+Text Label 8400 2300 0    50   ~ 0
+pa10
+Text Label 8400 2400 0    50   ~ 0
+pa09
+Text Label 8400 2100 0    50   ~ 0
+pb11
+Text Label 8400 2200 0    50   ~ 0
+pb10
+Text Label 8400 1900 0    50   ~ 0
+pb13
+Text Label 8400 2000 0    50   ~ 0
+pb12
+Text Label 8400 2700 0    50   ~ 0
+pa07
+Text Label 8400 2900 0    50   ~ 0
+pa08
+Text Label 8400 2600 0    50   ~ 0
+pa06
+Text Label 8400 2800 0    50   ~ 0
+pa05
+Text Label 8400 2500 0    50   ~ 0
+pa04
+Text Label 7850 3100 2    50   ~ 0
+pb17
+Text Label 7850 2500 2    50   ~ 0
+pa20
+Text Label 7850 2100 2    50   ~ 0
+pb01
 $EndSCHEMATC

Commit message: Moved User LED from PB08 to PB09
 - Updated schematic
 - Rerouted trace
 - Updated silkscreen
Connections:
- net pb08: no longer D2.2 (A)
- net pb09: now also D2.2 (A)
Changed lines of the file:
@@
 pa14
 Text Label 5850 2300 2    50   ~ 0
-pb08
+pb09
 Text Label 5850 2400 2    50   ~ 0
 pb06

Commit message: Fix silkscreen for new pinout, add PTS636 3D model.
Parts:
- C13: footprint Resistor_SMD:R_0402_1005Metric -> Capacitor_SMD:C_0402_1005Metric
Changed lines of the file:
@@
 F 0 "C13" V 10450 1150 50  0000 C CNN
 F 1 "100n" V 10512 1150 50  0000 C CNN
-F 2 "Resistor_SMD:R_0402_1005Metric" H 10650 1150 50  0001 C CNN
+F 2 "Capacitor_SMD:C_0402_1005Metric" H 10650 1150 50  0001 C CNN
 F 3 "~" H 10650 1150 50  0001 C CNN
 	1    10650 1150

Commit message: move silkscreen around on the bottom, add gear logo, adjust copper text
Parts:
- added LOGO1: Logo_Open_Hardware_Small, greenpill:OSHW-Symbol_4x4.5mm_SilkScreen, symbol Graphic:Logo_Open_Hardware_Small
Changed lines of the file:
@@
 	1150 1250 1150 1050
 Connection ~ 1150 1050
-$Comp
-L Graphic:Logo_Open_Hardware_Small #LOGO1
-U 1 1 5F548A14
-P 4750 3300
-F 0 "#LOGO1" H 4750 3575 50  0001 C CNN
-F 1 "Logo_Open_Hardware_Small" H 4750 3075 50  0001 C CNN
-F 2 "" H 4750 3300 50  0001 C CNN
-F 3 "~" H 4750 3300 50  0001 C CNN
-	1    4750 3300
-	1    0    0    -1
-$EndComp
 Text Label 7850 2800 2    50   ~ 0
 pa27
@@
 Text Label 7850 2100 2    50   ~ 0
 pb01
+$Comp
+L Graphic:Logo_Open_Hardware_Small LOGO1
+U 1 1 5F6303FA
+P 5150 3050
+F 0 "LOGO1" H 5150 3325 50  0001 C CNN
+F 1 "Logo_Open_Hardware_Small" H 5150 2825 50  0001 C CNN
+F 2 "greenpill:OSHW-Symbol_4x4.5mm_SilkScreen" H 5150 3050 50  0001 C CNN
+F 3 "~" H 5150 3050 50  0001 C CNN
+	1    5150 3050
+	1    0    0    -1
+$EndComp
 $EndSCHEMATC
